File: IMP_nano/IMP_nano.kicad_sch (KiCad schematic)
At the start: 39 parts, among them J1 KF301, J2 SH1.04PIN, Q1 BC847, Q2 AO3400A, SW1 SW_DPST_x2, SW2 SW_DIP_x04, U1 STM32L051C8T6

Commit message: Schematic cleaning, reviewed be me
Connections:
- net M_PB13 is gone; now on net M_PB12: R10.2, SW2.3, U1.26 (PB13)
Other:
- company: (none) -> Designed by Volodimir Martynov
- title: (none) -> IMP_NANO
- moved on the sheet: R10, R11, R12, R8, SW2

Commit message: Shematic update by VM
Iniciation shrmatic editing
Parts:
- removed BT1: MN21, IMP_LIB:BAT_BH23APC, symbol IMP_LIB_SYM:BH23APC
- removed C5: 3300u, Capacitor_THT:CP_Radial_D13.0mm_P5.00mm, symbol Device:C_Polarized
- removed D1: 1N5824, Diode_SMD:D_SMA, symbol Diode:1N5822
- removed J1: KF301, IMP_LIB:HANDSON_KF301-2P, symbol Connector:Conn_01x02_Pin
- removed Q1: BC847, Package_TO_SOT_SMD:SOT-23, symbol Transistor_BJT:BC847
- removed Q2: AO3400A, Package_TO_SOT_SMD:SOT-23, symbol Transistor_FET:AO3400A
- removed R3, R4: 120R, Resistor_SMD:R_0201_0603Metric, symbol Device:R
- removed R5: 10k, Resistor_SMD:R_0201_0603Metric, symbol Device:R
- removed R7: 240R, IMP_LIB:RESC6432X90N, symbol Device:R
Other:
- note removed: "Pull-down (For deafult statement OFF)"
- note removed: "R = 12 В / 0.05 А(I_charge) ≈ 240 Ω"
- note removed: "R= VCC/ gpio_max_A"
